Commit message: robot_agv

File: urdf/robot_agv.urdf (robot description, URDF)
Before this commit: robot robot_agv, 7 links, 6 joints
Links:
- link link_camera: mass 0.00436250529984365 -> 0.00436250529984944
Joints:
- joint joint_SP: origin xyz=-0.106268560503509 -0.0229661476240984 -0.0744999999999773 rpy=0 0 -0.146106215322719 -> xyz=-0.085146446610614 -0.100000000000507 -0.0229999999933239 rpy=-1.57079632681722 -0.146106215270251 0
- joint joint_ST: origin xyz=-0.106268560503509 -0.0229661476240978 0.125500000000023 rpy=0 0 0.418974378678853 -> xyz=-0.0851464466106142 0.0999999999994928 -0.0229999999977417 rpy=-1.57079632681907 0.418974378731321 0
- joint joint_TP: origin xyz=0.0500243327153047 -0.0229661476240979 -0.0744999999999778 rpy=0 0 0 -> xyz=0.0711464466081992 -0.100000000000508 -0.0230000000015247 rpy=-1.57079632681698 0 0
- joint joint_TT: origin xyz=0.0500243327153045 -0.0229661476240979 0.125500000000023 rpy=0 0 0 -> xyz=0.071146446608199 0.0999999999994926 -0.023000000005942 rpy=-1.57079632681698 0 0
- joint joint_camera: origin xyz=0.0906778861058987 -0.0218736065266276 0.0267016521433842 rpy=0 0 1.5707963267949 -> xyz=0.111799999998736 0.00120165214283002 -0.0240925411033633 rpy=1.5707963267949 1.5707963267949 0
- joint joint_lidar: origin xyz=0 -0.0749661476240983 0.0275000000000219 rpy=1.5707963267949 0 0 -> xyz=0.0211221138956228 0.00200000000064026 0.0289999999988475 rpy=0 0 0

Commit message: robot_agv

File: urdf/robot_agv.urdf (robot description, URDF)
Before this commit: robot robot_agv, 7 links, 6 joints
Links:
- link link_camera: mass 0.00436250529984944 -> 0.00436250529984364
Joints:
- joint joint_camera: origin xyz=0.111799999998736 0.00120165214283002 -0.0240925411033633 rpy=1.5707963267949 1.5707963267949 0 -> xyz=0.111799999998736 0.00120165214283002 -0.0240925411033633 rpy=-1.57079632681698 0 0
